Commit message: resolve gazebo_ros2_control plugin crash by simplifying URDF

File: src/fairino_description/urdf/fairino3_v6.urdf.xacro (robot description, xacro)
@@ -27,19 +27,19 @@
       <geometry>
         <mesh
-          filename="package://fairino_description/meshes/fairino3_v6/base_link.STL" />
-      </geometry>
-      <material
-        name="">
-        <color
-          rgba="0.89804 0.91765 0.92941 1" />
-      </material>
-    </visual>
-    <collision>
-      <origin
-        xyz="0 0 0"
-        rpy="0 0 0" />
-      <geometry>
-        <mesh
-          filename="package://fairino_description/meshes/fairino3_v6/base_link.STL" />
+          filename="file:///$(find fairino_description)/meshes/fairino3_v6/base_link.STL" />
+      </geometry>
+      <material
+        name="">
+        <color
+          rgba="0.89804 0.91765 0.92941 1" />
+      </material>
+    </visual>
+    <collision>
+      <origin
+        xyz="0 0 0"
+        rpy="0 0 0" />
+      <geometry>
+        <mesh
+          filename="file:///$(find fairino_description)/meshes/fairino3_v6/base_link.STL" />
       </geometry>
     </collision>
@@ -67,19 +67,19 @@
       <geometry>
         <mesh
-          filename="package://fairino_description/meshes/fairino3_v6/shoulder_link.STL" />
-      </geometry>
-      <material
-        name="">
-        <color
-          rgba="0.89804 0.91765 0.92941 1" />
-      </material>
-    </visual>
-    <collision>
-      <origin
-        xyz="0 0 0"
-        rpy="0 0 0" />
-      <geometry>
-        <mesh
-          filename="package://fairino_description/meshes/fairino3_v6/shoulder_link.STL" />
+          filename="file:///$(find fairino_description)/meshes/fairino3_v6/shoulder_link.STL" />
+      </geometry>
+      <material
+        name="">
+        <color
+          rgba="0.89804 0.91765 0.92941 1" />
+      </material>
+    </visual>
+    <collision>
+      <origin
+        xyz="0 0 0"
+        rpy="0 0 0" />
+      <geometry>
+        <mesh
+         filename="file:///$(find fairino_description)/meshes/fairino3_v6/shoulder_link.STL" />
       </geometry>
     </collision>
@@ -136,19 +136,19 @@
       <geometry>
         <mesh
-          filename="package://fairino_description/meshes/fairino3_v6/upperarm_link.STL" />
-      </geometry>
-      <material
-        name="">
-        <color
-          rgba="0.89804 0.91765 0.92941 1" />
-      </material>
-    </visual>
-    <collision>
-      <origin
-        xyz="0 0 0"
-        rpy="0 0 0" />
-      <geometry>
-        <mesh
-          filename="package://fairino_description/meshes/fairino3_v6/upperarm_link.STL" />
+         filename="file:///$(find fairino_description)/meshes/fairino3_v6/upperarm_link.STL" />
+      </geometry>
+      <material
+        name="">
+        <color
+          rgba="0.89804 0.91765 0.92941 1" />
+      </material>
+    </visual>
+    <collision>
+      <origin
+        xyz="0 0 0"
+        rpy="0 0 0" />
+      <geometry>
+        <mesh
+         filename="file:///$(find fairino_description)/meshes/fairino3_v6/upperarm_link.STL" />
       </geometry>
     </collision>
@@ -205,19 +205,19 @@
       <geometry>
         <mesh
-          filename="package://fairino_description/meshes/fairino3_v6/forearm_link.STL" />
-      </geometry>
-      <material
-        name="">
-        <color
-          rgba="0.89804 0.91765 0.92941 1" />
-      </material>
-    </visual>
-    <collision>
-      <origin
-        xyz="0 0 0"
-        rpy="0 0 0" />
-      <geometry>
-        <mesh
-          filename="package://fairino_description/meshes/fairino3_v6/forearm_link.STL" />
+          filename="file:///$(find fairino_description)/meshes/fairino3_v6/forearm_link.STL" />
+      </geometry>
+      <material
+        name="">
+        <color
+          rgba="0.89804 0.91765 0.92941 1" />
+      </material>
+    </visual>
+    <collision>
+      <origin
+        xyz="0 0 0"
+        rpy="0 0 0" />
+      <geometry>
+        <mesh
+         filename="file:///$(find fairino_description)/meshes/fairino3_v6/forearm_link.STL" />
       </geometry>
     </collision>
@@ -274,19 +274,19 @@
       <geometry>
         <mesh
-          filename="package://fairino_description/meshes/fairino3_v6/wrist1_link.STL" />
-      </geometry>
-      <material
-        name="">
-        <color
-          rgba="0.89804 0.91765 0.92941 1" />
-      </material>
-    </visual>
-    <collision>
-      <origin
-        xyz="0 0 0"
-        rpy="0 0 0" />
-      <geometry>
-        <mesh
-          filename="package://fairino_description/meshes/fairino3_v6/wrist1_link.STL" />
+        filename="file:///$(find fairino_description)/meshes/fairino3_v6/wrist1_link.STL" />
+      </geometry>
+      <material
+        name="">
+        <color
+          rgba="0.89804 0.91765 0.92941 1" />
+      </material>
+    </visual>
+    <collision>
+      <origin
+        xyz="0 0 0"
+        rpy="0 0 0" />
+      <geometry>
+        <mesh
+         filename="file:///$(find fairino_description)/meshes/fairino3_v6/wrist1_link.STL" />
       </geometry>
     </collision>
@@ -343,19 +343,19 @@
       <geometry>
         <mesh
-          filename="package://fairino_description/meshes/fairino3_v6/wrist2_link.STL" />
-      </geometry>
-      <material
-        name="">
-        <color
-          rgba="0.89804 0.91765 0.92941 1" />
-      </material>
-    </visual>
-    <collision>
-      <origin
-        xyz="0 0 0"
-        rpy="0 0 0" />
-      <geometry>
-        <mesh
-          filename="package://fairino_description/meshes/fairino3_v6/wrist2_link.STL" />
+          filename="file:///$(find fairino_description)/meshes/fairino3_v6/wrist2_link.STL" />
+      </geometry>
+      <material
+        name="">
+        <color
+          rgba="0.89804 0.91765 0.92941 1" />
+      </material>
+    </visual>
+    <collision>
+      <origin
+        xyz="0 0 0"
+        rpy="0 0 0" />
+      <geometry>
+        <mesh
+         filename="file:///$(find fairino_description)/meshes/fairino3_v6/wrist2_link.STL" />
       </geometry>
     </collision>
@@ -412,19 +412,19 @@
       <geometry>
         <mesh
-          filename="package://fairino_description/meshes/fairino3_v6/wrist3_link.STL" />
-      </geometry>
-      <material
-        name="">
-        <color
-          rgba="0.89804 0.91765 0.92941 1" />
-      </material>
-    </visual>
-    <collision>
-      <origin
-        xyz="0 0 0"
-        rpy="0 0 0" />
-      <geometry>
-        <mesh
-          filename="package://fairino_description/meshes/fairino3_v6/wrist3_link.STL" />
+          filename="file:///$(find fairino_description)/meshes/fairino3_v6/wrist3_link.STL" />
+      </geometry>
+      <material
+        name="">
+        <color
+          rgba="0.89804 0.91765 0.92941 1" />
+      </material>
+    </visual>
+    <collision>
+      <origin
+        xyz="0 0 0"
+        rpy="0 0 0" />
+      <geometry>
+        <mesh
+          filename="file:///$(find fairino_description)/meshes/fairino3_v6/wrist3_link.STL" />
       </geometry>
     </collision>
@@ -459,3 +459,116 @@
       k_velocity="10" />
   </joint>
+  <transmission name="trans_j1">
+  <type>transmission_interface/SimpleTransmission</type>
+  <joint name="j1">
+   <hardwareInterface>hardware_interface/PositionJointInterface</hardwareInterface>
+  </joint>
+  <actuator name="motor1">
+   <hardwareInterface>hardware_interface/PositionJointInterface</hardwareInterface>
+   <mechanicalReduction>1</mechanicalReduction>
+  </actuator>
+ </transmission>
+ <transmission name="trans_j2">
+  <type>transmission_interface/SimpleTransmission</type>
+  <joint name="j2">
+   <hardwareInterface>hardware_interface/PositionJointInterface</hardwareInterface>
+  </joint>
+  <actuator name="motor2">
+   <hardwareInterface>hardware_interface/PositionJointInterface</hardwareInterface>
+   <mechanicalReduction>1</mechanicalReduction>
+  </actuator>
+ </transmission>
+ <transmission name="trans_j3">
+  <type>transmission_interface/SimpleTransmission</type>
+  <joint name="j3">
+   <hardwareInterface>hardware_interface/PositionJointInterface</hardwareInterface>
+  </joint>
+  <actuator name="motor3">
+   <hardwareInterface>hardware_interface/PositionJointInterface</hardwareInterface>
+   <mechanicalReduction>1</mechanicalReduction>
+  </actuator>
+ </transmission>
+ <transmission name="trans_j4">
+  <type>transmission_interface/SimpleTransmission</type>
+  <joint name="j4">
+   <hardwareInterface>hardware_interface/PositionJointInterface</hardwareInterface>
+  </joint>
+  <actuator name="motor4">
+   <hardwareInterface>hardware_interface/PositionJointInterface</hardwareInterface>
+   <mechanicalReduction>1</mechanicalReduction>
+  </actuator>
+ </transmission>
+ <transmission name="trans_j5">
+  <type>transmission_interface/SimpleTransmission</type>
+  <joint name="j5">
+   <hardwareInterface>hardware_interface/PositionJointInterface</hardwareInterface>
+  </joint>
+  <actuator name="motor5">
+   <hardwareInterface>hardware_interface/PositionJointInterface</hardwareInterface>
+   <mechanicalReduction>1</mechanicalReduction>
+  </actuator>
+ </transmission>
+ <transmission name="trans_j6">
+  <type>transmission_interface/SimpleTransmission</type>
+  <joint name="j6">
+   <hardwareInterface>hardware_interface/PositionJointInterface</hardwareInterface>
+  </joint>
+  <actuator name="motor6">
+   <hardwareInterface>hardware_interface/PositionJointInterface</hardwareInterface>
+   <mechanicalReduction>1</mechanicalReduction>
+  </actuator>
+ </transmission>
+ <ros2_control name="GazeboSystem" type="system">
+      <hardware>
+        <plugin>gazebo_ros2_control/GazeboSystem</plugin>
+      </hardware>
+    <joint name="j1">
+      <command_interface name="position">
+        <param name="min">-1.57</param>
+        <param name="max">1.57</param>
+      </command_interface>
+        <state_interface name="position"/>
+        <state_interface name="velocity"/>
+    </joint>
+    <joint name="j2">
+      <command_interface name="position">
+        <param name="min">-1.57</param>
+        <param name="max">1.57</param>
+      </command_interface>
+      <state_interface name="position"/>
+      <state_interface name="velocity"/>
+    </joint>
+    <joint name="j3">
+      <command_interface name="position">
+        <param name="min">-1.57</param>
+        <param name="max">1.57</param>
+      </command_interface>
+      <state_interface name="position"/>
+      <state_interface name="velocity"/>
+    </joint>
+    <joint name="j4">
+      <command_interface name="position">
+        <param name="min">-1.57</param>
+        <param name="max">1.57</param>
+      </command_interface>
+      <state_interface name="position"/>
+      <state_interface name="velocity"/>
+    </joint>
+    <joint name="j5">
+      <command_interface name="position">
+        <param name="min">-1.57</param>
+        <param name="max">1.57</param>
+      </command_interface>
+      <state_interface name="position"/>
+      <state_interface name="velocity"/>
+    </joint>
+    <joint name="j6">
+        <command_interface name="position">
+            <param name="min">-1.57</param>
+            <param name="max">1.57</param>
+        </command_interface>
+        <state_interface name="position"/>
+        <state_interface name="velocity"/>
+      </joint>
+ </ros2_control>
 </robot>

File: src/fairino_description/urdf_dual_arms/fairino3_dual_arms.urdf.xacro (robot description, xacro)
@@ -49,57 +49,57 @@
   <!-- ros2_control (single system with 12 joints) -->
   <ros2_control name="dual_arms_system" type="system">
-    <joint name="${left_prefix}joint1">
+    <hardware>
+      <plugin>gazebo_ros2_control/GazeboSystem</plugin>
+    </hardware>
+    <!-- Left arm joints -->
+    <joint name="${left_prefix}j1">
       <command_interface name="position"/>
       <state_interface name="position"/>
     </joint>
-    <joint name="${left_prefix}joint2">
+    <joint name="${left_prefix}j2">
       <command_interface name="position"/>
       <state_interface name="position"/>
     </joint>
-    <joint name="${left_prefix}joint3">
+    <joint name="${left_prefix}j3">
       <command_interface name="position"/>
       <state_interface name="position"/>
     </joint>
-    <joint name="${left_prefix}joint4">
+    <joint name="${left_prefix}j4">
       <command_interface name="position"/>
       <state_interface name="position"/>
     </joint>
-    <joint name="${left_prefix}joint5">
+    <joint name="${left_prefix}j5">
       <command_interface name="position"/>
       <state_interface name="position"/>
     </joint>
-    <joint name="${left_prefix}joint6">
+    <joint name="${left_prefix}j6">
       <command_interface name="position"/>
       <state_interface name="position"/>
     </joint>
-    <joint name="${right_prefix}joint1">
+    <!-- Right arm joints -->
+    <joint name="${right_prefix}j1">
       <command_interface name="position"/>
       <state_interface name="position"/>
     </joint>
-    <joint name="${right_prefix}joint2">
+    <joint name="${right_prefix}j2">
       <command_interface name="position"/>
       <state_interface name="position"/>
     </joint>
-    <joint name="${right_prefix}joint3">
+    <joint name="${right_prefix}j3">
       <command_interface name="position"/>
       <state_interface name="position"/>
     </joint>
-    <joint name="${right_prefix}joint4">
+    <joint name="${right_prefix}j4">
       <command_interface name="position"/>
       <state_interface name="position"/>
     </joint>
-    <joint name="${right_prefix}joint5">
+    <joint name="${right_prefix}j5">
       <command_interface name="position"/>
       <state_interface name="position"/>
     </joint>
-    <joint name="${right_prefix}joint6">
+    <joint name="${right_prefix}j6">
       <command_interface name="position"/>
       <state_interface name="position"/>
     </joint>
   </ros2_control>
-  <!-- <gazebo>
-    <plugin filename="ign_ros2_control-system" name="ign_ros2_control::IgnitionROS2ControlPlugin">
-      <parameters>${ros2_controllers_file}</parameters>
-    </plugin>
-  </gazebo> -->
 </robot>

File: src/fairino_description/urdf_dual_arms/fairino3_v6_robot.prefixed.urdf.xacro (robot description, xacro)
@@ -24,19 +24,19 @@
       <geometry>
         <mesh
-          filename="package://fairino_description/meshes/fairino3_v6/base_link.STL" />
-      </geometry>
-      <material
-        name="">
-        <color
-          rgba="0.89804 0.91765 0.92941 1" />
-      </material>
-    </visual>
-    <collision>
-      <origin
-        xyz="0 0 0"
-        rpy="0 0 0" />
-      <geometry>
-        <mesh
-          filename="package://fairino_description/meshes/fairino3_v6/base_link.STL" />
+          filename="file:///$(find fairino_description)/meshes/fairino3_v6/base_link.STL" />
+      </geometry>
+      <material
+        name="">
+        <color
+          rgba="0.89804 0.91765 0.92941 1" />
+      </material>
+    </visual>
+    <collision>
+      <origin
+        xyz="0 0 0"
+        rpy="0 0 0" />
+      <geometry>
+        <mesh
+          filename="file:///$(find fairino_description)/meshes/fairino3_v6/base_link.STL" />
       </geometry>
     </collision>
@@ -64,19 +64,19 @@
       <geometry>
         <mesh
-          filename="package://fairino_description/meshes/fairino3_v6/shoulder_link.STL" />
-      </geometry>
-      <material
-        name="">
-        <color
-          rgba="0.89804 0.91765 0.92941 1" />
-      </material>
-    </visual>
-    <collision>
-      <origin
-        xyz="0 0 0"
-        rpy="0 0 0" />
-      <geometry>
-        <mesh
-          filename="package://fairino_description/meshes/fairino3_v6/shoulder_link.STL" />
+          filename="file:///$(find fairino_description)/meshes/fairino3_v6/shoulder_link.STL" />
+      </geometry>
+      <material
+        name="">
+        <color
+          rgba="0.89804 0.91765 0.92941 1" />
+      </material>
+    </visual>
+    <collision>
+      <origin
+        xyz="0 0 0"
+        rpy="0 0 0" />
+      <geometry>
+        <mesh
+          filename="file:///$(find fairino_description)/meshes/fairino3_v6/shoulder_link.STL" />
       </geometry>
     </collision>
@@ -133,19 +133,19 @@
       <geometry>
         <mesh
-          filename="package://fairino_description/meshes/fairino3_v6/upperarm_link.STL" />
-      </geometry>
-      <material
-        name="">
-        <color
-          rgba="0.89804 0.91765 0.92941 1" />
-      </material>
-    </visual>
-    <collision>
-      <origin
-        xyz="0 0 0"
-        rpy="0 0 0" />
-      <geometry>
-        <mesh
-          filename="package://fairino_description/meshes/fairino3_v6/upperarm_link.STL" />
+          filename="file:///$(find fairino_description)/meshes/fairino3_v6/upperarm_link.STL" />
+      </geometry>
+      <material
+        name="">
+        <color
+          rgba="0.89804 0.91765 0.92941 1" />
+      </material>
+    </visual>
+    <collision>
+      <origin
+        xyz="0 0 0"
+        rpy="0 0 0" />
+      <geometry>
+        <mesh
+          filename="file:///$(find fairino_description)/meshes/fairino3_v6/upperarm_link.STL" />
       </geometry>
     </collision>
@@ -202,19 +202,19 @@
       <geometry>
         <mesh
-          filename="package://fairino_description/meshes/fairino3_v6/forearm_link.STL" />
-      </geometry>
-      <material
-        name="">
-        <color
-          rgba="0.89804 0.91765 0.92941 1" />
-      </material>
-    </visual>
-    <collision>
-      <origin
-        xyz="0 0 0"
-        rpy="0 0 0" />
-      <geometry>
-        <mesh
-          filename="package://fairino_description/meshes/fairino3_v6/forearm_link.STL" />
+          filename="file:///$(find fairino_description)/meshes/fairino3_v6/forearm_link.STL" />
+      </geometry>
+      <material
+        name="">
+        <color
+          rgba="0.89804 0.91765 0.92941 1" />
+      </material>
+    </visual>
+    <collision>
+      <origin
+        xyz="0 0 0"
+        rpy="0 0 0" />
+      <geometry>
+        <mesh
+          filename="package://fairino_description)/meshes/fairino3_v6/forearm_link.STL" />
       </geometry>
     </collision>
@@ -271,19 +271,19 @@
       <geometry>
         <mesh
-          filename="package://fairino_description/meshes/fairino3_v6/wrist1_link.STL" />
-      </geometry>
-      <material
-        name="">
-        <color
-          rgba="0.89804 0.91765 0.92941 1" />
-      </material>
-    </visual>
-    <collision>
-      <origin
-        xyz="0 0 0"
-        rpy="0 0 0" />
-      <geometry>
-        <mesh
-          filename="package://fairino_description/meshes/fairino3_v6/wrist1_link.STL" />
+          filename="file:///$(find fairino_description)/meshes/fairino3_v6/wrist1_link.STL" />
+      </geometry>
+      <material
+        name="">
+        <color
+          rgba="0.89804 0.91765 0.92941 1" />
+      </material>
+    </visual>
+    <collision>
+      <origin
+        xyz="0 0 0"
+        rpy="0 0 0" />
+      <geometry>
+        <mesh
+          filename="file:///$(find fairino_description)/meshes/fairino3_v6/wrist1_link.STL" />
       </geometry>
     </collision>
@@ -340,19 +340,19 @@
       <geometry>
         <mesh
-          filename="package://fairino_description/meshes/fairino3_v6/wrist2_link.STL" />
-      </geometry>
-      <material
-        name="">
-        <color
-          rgba="0.89804 0.91765 0.92941 1" />
-      </material>
-    </visual>
-    <collision>
-      <origin
-        xyz="0 0 0"
-        rpy="0 0 0" />
-      <geometry>
-        <mesh
-          filename="package://fairino_description/meshes/fairino3_v6/wrist2_link.STL" />
+          filename="file:///$(find fairino_description)/meshes/fairino3_v6/wrist2_link.STL" />
+      </geometry>
+      <material
+        name="">
+        <color
+          rgba="0.89804 0.91765 0.92941 1" />
+      </material>
+    </visual>
+    <collision>
+      <origin
+        xyz="0 0 0"
+        rpy="0 0 0" />
+      <geometry>
+        <mesh
+          filename="file:///$(find fairino_description)/meshes/fairino3_v6/wrist2_link.STL" />
       </geometry>
     </collision>
@@ -409,19 +409,19 @@
       <geometry>
         <mesh
-          filename="package://fairino_description/meshes/fairino3_v6/wrist3_link.STL" />
-      </geometry>
-      <material
-        name="">
-        <color
-          rgba="0.89804 0.91765 0.92941 1" />
-      </material>
-    </visual>
-    <collision>
-      <origin
-        xyz="0 0 0"
-        rpy="0 0 0" />
-      <geometry>
-        <mesh
-          filename="package://fairino_description/meshes/fairino3_v6/wrist3_link.STL" />
+          filename="file:///$(find fairino_description)/meshes/fairino3_v6/wrist3_link.STL" />
+      </geometry>
+      <material
+        name="">
+        <color
+          rgba="0.89804 0.91765 0.92941 1" />
+      </material>
+    </visual>
+    <collision>
+      <origin
+        xyz="0 0 0"
+        rpy="0 0 0" />
+      <geometry>
+        <mesh
+          filename="file:///$(find fairino_description)/meshes/fairino3_v6/wrist3_link.STL" />
       </geometry>
     </collision>
