Commit message: dual_arm_position_controller remains unconfigured due to wrong URDF interface declaration

File: src/fairino_description/urdf_dual_arms/fairino3_dual_arms.urdf.xacro (robot description, xacro)
@@ -5,7 +5,7 @@
   <xacro:arg name="arm_spacing" default="0.75"/>
   <xacro:arg name="initial_positions_file"
-           default="$(find fairino_description)/urdf_dual_arms/initial_positions.yaml"/>
+           default="$(find fairino_description)/config/initial_positions.yaml"/>
   <xacro:arg name="ros2_controllers_file"
-           default="$(find fairino_description)/urdf_dual_arms/ros2_controllers.yaml"/>
+           default="$(find fairino_description)/config/ros2_controllers.yaml"/>
   <xacro:arg name="floor_size_x" default="4.0"/>
   <xacro:arg name="floor_size_y" default="4.0"/>
@@ -49,57 +49,66 @@
   <!-- ros2_control (single system with 12 joints) -->
   <ros2_control name="dual_arms_system" type="system">
-    <hardware>
-      <plugin>gazebo_ros2_control/GazeboSystem</plugin>
-    </hardware>
-    <!-- Left arm joints -->
-    <joint name="${left_prefix}j1">
-      <command_interface name="position"/>
-      <state_interface name="position"/>
-    </joint>
-    <joint name="${left_prefix}j2">
-      <command_interface name="position"/>
-      <state_interface name="position"/>
-    </joint>
-    <joint name="${left_prefix}j3">
-      <command_interface name="position"/>
-      <state_interface name="position"/>
-    </joint>
-    <joint name="${left_prefix}j4">
-      <command_interface name="position"/>
-      <state_interface name="position"/>
-    </joint>
-    <joint name="${left_prefix}j5">
-      <command_interface name="position"/>
-      <state_interface name="position"/>
-    </joint>
-    <joint name="${left_prefix}j6">
-      <command_interface name="position"/>
-      <state_interface name="position"/>
-    </joint>
-    <!-- Right arm joints -->
-    <joint name="${right_prefix}j1">
-      <command_interface name="position"/>
-      <state_interface name="position"/>
-    </joint>
-    <joint name="${right_prefix}j2">
-      <command_interface name="position"/>
-      <state_interface name="position"/>
-    </joint>
-    <joint name="${right_prefix}j3">
-      <command_interface name="position"/>
-      <state_interface name="position"/>
-    </joint>
-    <joint name="${right_prefix}j4">
-      <command_interface name="position"/>
-      <state_interface name="position"/>
-    </joint>
-    <joint name="${right_prefix}j5">
-      <command_interface name="position"/>
-      <state_interface name="position"/>
-    </joint>
-    <joint name="${right_prefix}j6">
-      <command_interface name="position"/>
-      <state_interface name="position"/>
-    </joint>
+  <hardware>
+    <plugin>gazebo_ros2_control/GazeboSystem</plugin>
+  </hardware>
+  <!-- Left arm joints -->
+  <joint name="${left_prefix}joint1">
+    <command_interfaces>
+      <position/>
+    </command_interfaces>
+    <state_interfaces>
+      <position/>
+    </state_interfaces>
+  </joint>
+  <joint name="${left_prefix}joint2">
+    <command_interfaces><position/></command_interfaces>
+    <state_interfaces><position/></state_interfaces>
+  </joint>
+  <joint name="${left_prefix}joint3">
+    <command_interfaces><position/></command_interfaces>
+    <state_interfaces><position/></state_interfaces>
+  </joint>
+  <joint name="${left_prefix}joint4">
+    <command_interfaces><position/></command_interfaces>
+    <state_interfaces><position/></state_interfaces>
+  </joint>
+  <joint name="${left_prefix}joint5">
+    <command_interfaces><position/></command_interfaces>
+    <state_interfaces><position/></state_interfaces>
+  </joint>
+  <joint name="${left_prefix}joint6">
+    <command_interfaces><position/></command_interfaces>
+    <state_interfaces><position/></state_interfaces>
+  </joint>
+  <!-- Right arm joints -->
+  <joint name="${right_prefix}joint1">
+    <command_interfaces><position/></command_interfaces>
+    <state_interfaces><position/></state_interfaces>
+  </joint>
+  <joint name="${right_prefix}joint2">
+    <command_interfaces><position/></command_interfaces>
+    <state_interfaces><position/></state_interfaces>
+  </joint>
+  <joint name="${right_prefix}joint3">
+    <command_interfaces><position/></command_interfaces>
+    <state_interfaces><position/></state_interfaces>
+  </joint>
+  <joint name="${right_prefix}joint4">
+    <command_interfaces><position/></command_interfaces>
+    <state_interfaces><position/></state_interfaces>
+  </joint>
+  <joint name="${right_prefix}joint5">
+    <command_interfaces><position/></command_interfaces>
+    <state_interfaces><position/></state_interfaces>
+  </joint>
+  <joint name="${right_prefix}joint6">
+    <command_interfaces><position/></command_interfaces>
+    <state_interfaces><position/></state_interfaces>
+  </joint>
   </ros2_control>
+  <gazebo>
+    <plugin name="gazebo_ros2_control" filename="libgazebo_ros2_control.so">
+      <parameters>$(find fairino_description)/config/ros2_controllers.yaml</parameters>
+    </plugin>
+  </gazebo>
 </robot>

Commit message: dual-arm controller YAML and usage commands, Gazebo load successful

File: src/fairino_description/urdf_dual_arms/fairino3_dual_arms.urdf.xacro (robot description, xacro)
@@ -54,55 +54,76 @@
   <!-- Left arm joints -->
   <joint name="${left_prefix}joint1">
-    <command_interfaces>
-      <position/>
-    </command_interfaces>
-    <state_interfaces>
-      <position/>
-    </state_interfaces>
+    <command_interface name="position" />
+    <state_interface name="position" />
+    <state_interface name="velocity" />
+    <state_interface name="effort" />
   </joint>
   <joint name="${left_prefix}joint2">
-    <command_interfaces><position/></command_interfaces>
-    <state_interfaces><position/></state_interfaces>
+    <command_interface name="position" />
+    <state_interface name="position" />
+    <state_interface name="velocity" />
+    <state_interface name="effort" />
   </joint>
   <joint name="${left_prefix}joint3">
     <command_interfaces><position/></command_interfaces>
-    <state_interfaces><position/></state_interfaces>
+    <command_interface name="position" />
+    <state_interface name="position" />
+    <state_interface name="velocity" />
+    <state_interface name="effort" />
   </joint>
   <joint name="${left_prefix}joint4">
-    <command_interfaces><position/></command_interfaces>
-    <state_interfaces><position/></state_interfaces>
+    <command_interface name="position" />
+    <state_interface name="position" />
+    <state_interface name="velocity" />
+    <state_interface name="effort" />
   </joint>
   <joint name="${left_prefix}joint5">
-    <command_interfaces><position/></command_interfaces>
-    <state_interfaces><position/></state_interfaces>
+    <command_interface name="position" />
+    <state_interface name="position" />
+    <state_interface name="velocity" />
+    <state_interface name="effort" />
   </joint>
   <joint name="${left_prefix}joint6">
-    <command_interfaces><position/></command_interfaces>
-    <state_interfaces><position/></state_interfaces>
+    <command_interface name="position" />
+    <state_interface name="position" />
+    <state_interface name="velocity" />
+    <state_interface name="effort" />
   </joint>
   <!-- Right arm joints -->
   <joint name="${right_prefix}joint1">
-    <command_interfaces><position/></command_interfaces>
-    <state_interfaces><position/></state_interfaces>
+    <command_interface name="position" />
+    <state_interface name="position" />
+    <state_interface name="velocity" />
+    <state_interface name="effort" />
   </joint>
   <joint name="${right_prefix}joint2">
-    <command_interfaces><position/></command_interfaces>
-    <state_interfaces><position/></state_interfaces>
+    <command_interface name="position" />
+    <state_interface name="position" />
+    <state_interface name="velocity" />
+    <state_interface name="effort" />
   </joint>
   <joint name="${right_prefix}joint3">
-    <command_interfaces><position/></command_interfaces>
-    <state_interfaces><position/></state_interfaces>
+    <command_interface name="position" />
+    <state_interface name="position" />
+    <state_interface name="velocity" />
+    <state_interface name="effort" />
   </joint>
   <joint name="${right_prefix}joint4">
-    <command_interfaces><position/></command_interfaces>
-    <state_interfaces><position/></state_interfaces>
+    <command_interface name="position" />
+    <state_interface name="position" />
+    <state_interface name="velocity" />
+    <state_interface name="effort" />
   </joint>
   <joint name="${right_prefix}joint5">
-    <command_interfaces><position/></command_interfaces>
-    <state_interfaces><position/></state_interfaces>
+    <command_interface name="position" />
+    <state_interface name="position" />
+    <state_interface name="velocity" />
+    <state_interface name="effort" />
   </joint>
   <joint name="${right_prefix}joint6">
-    <command_interfaces><position/></command_interfaces>
-    <state_interfaces><position/></state_interfaces>
+    <command_interface name="position" />
+    <state_interface name="position" />
+    <state_interface name="velocity" />
+    <state_interface name="effort" />
   </joint>
   </ros2_control>

File: src/fairino_description/urdf_dual_arms/fairino3_v6_robot.prefixed.urdf.xacro (robot description, xacro)
@@ -24,22 +24,26 @@
       <geometry>
         <mesh
-          filename="file:///$(find fairino_description)/meshes/fairino3_v6/base_link.STL" />
-      </geometry>
-      <material
-        name="">
-        <color
-          rgba="0.89804 0.91765 0.92941 1" />
-      </material>
-    </visual>
-    <collision>
-      <origin
-        xyz="0 0 0"
-        rpy="0 0 0" />
-      <geometry>
-        <mesh
-          filename="file:///$(find fairino_description)/meshes/fairino3_v6/base_link.STL" />
-      </geometry>
-    </collision>
-  </link>
+          filename="file://$(find fairino_description)/meshes/fairino3_v6/base_link.STL" />
+      </geometry>
+      <material
+        name="">
+        <color
+          rgba="0.89804 0.91765 0.92941 1" />
+      </material>
+    </visual>
+    <collision>
+      <origin
+        xyz="0 0 0"
+        rpy="0 0 0" />
+      <geometry>
+        <mesh
+          filename="file://$(find fairino_description)/meshes/fairino3_v6/base_link.STL" />
+      </geometry>
+    </collision>
+  </link>
+  <gazebo reference="${prefix}base_link">
+    <static>true</static>
+    <self_collide>false</self_collide>
+  </gazebo>
   <link
     name="${prefix}shoulder_link">
@@ -64,22 +68,23 @@
       <geometry>
         <mesh
-          filename="file:///$(find fairino_description)/meshes/fairino3_v6/shoulder_link.STL" />
-      </geometry>
-      <material
-        name="">
-        <color
-          rgba="0.89804 0.91765 0.92941 1" />
-      </material>
-    </visual>
-    <collision>
-      <origin
-        xyz="0 0 0"
-        rpy="0 0 0" />
-      <geometry>
-        <mesh
-          filename="file:///$(find fairino_description)/meshes/fairino3_v6/shoulder_link.STL" />
-      </geometry>
-    </collision>
-  </link>
+          filename="file://$(find fairino_description)/meshes/fairino3_v6/shoulder_link.STL" />
+      </geometry>
+      <material
+        name="">
+        <color
+          rgba="0.89804 0.91765 0.92941 1" />
+      </material>
+    </visual>
+    <collision>
+      <origin
+        xyz="0 0 0"
+        rpy="0 0 0" />
+      <geometry>
+        <mesh
+          filename="file://$(find fairino_description)/meshes/fairino3_v6/shoulder_link.STL" />
+      </geometry>
+    </collision>
+  </link>
+  <gazebo reference="${prefix}shoulder_link"><self_collide>false</self_collide></gazebo>
   <joint
     name="${prefix}joint1"
@@ -111,4 +116,14 @@
       k_velocity="10" />
   </joint>
+  <transmission name="${prefix}joint1_trans">
+    <type>transmission_interface/SimpleTransmission</type>
+    <joint name="${prefix}joint1">
+      <hardwareInterface>hardware_interface/PositionJointInterface</hardwareInterface>
+    </joint>
+    <actuator name="${prefix}joint1_motor">
+      <hardwareInterface>hardware_interface/PositionJointInterface</hardwareInterface>
+      <mechanicalReduction>1</mechanicalReduction>
+    </actuator>
+  </transmission>
   <link
     name="${prefix}upperarm_link">
@@ -133,22 +148,23 @@
       <geometry>
         <mesh
-          filename="file:///$(find fairino_description)/meshes/fairino3_v6/upperarm_link.STL" />
-      </geometry>
-      <material
-        name="">
-        <color
-          rgba="0.89804 0.91765 0.92941 1" />
-      </material>
-    </visual>
-    <collision>
-      <origin
-        xyz="0 0 0"
-        rpy="0 0 0" />
-      <geometry>
-        <mesh
-          filename="file:///$(find fairino_description)/meshes/fairino3_v6/upperarm_link.STL" />
-      </geometry>
-    </collision>
-  </link>
+          filename="file://$(find fairino_description)/meshes/fairino3_v6/upperarm_link.STL" />
+      </geometry>
+      <material
+        name="">
+        <color
+          rgba="0.89804 0.91765 0.92941 1" />
+      </material>
+    </visual>
+    <collision>
+      <origin
+        xyz="0 0 0"
+        rpy="0 0 0" />
+      <geometry>
+        <mesh
+          filename="file://$(find fairino_description)/meshes/fairino3_v6/upperarm_link.STL" />
+      </geometry>
+    </collision>
+  </link>
+  <gazebo reference="${prefix}upperarm_link"><self_collide>false</self_collide></gazebo>
   <joint
     name="${prefix}joint2"
@@ -180,4 +196,14 @@
       k_velocity="10" />
   </joint>
+  <transmission name="${prefix}joint2_trans">
+    <type>transmission_interface/SimpleTransmission</type>
+    <joint name="${prefix}joint2">
+      <hardwareInterface>hardware_interface/PositionJointInterface</hardwareInterface>
+    </joint>
+    <actuator name="${prefix}joint2_motor">
+      <hardwareInterface>hardware_interface/PositionJointInterface</hardwareInterface>
+      <mechanicalReduction>1</mechanicalReduction>
+    </actuator>
+  </transmission>
   <link
     name="${prefix}forearm_link">
@@ -202,22 +228,23 @@
       <geometry>
         <mesh
-          filename="file:///$(find fairino_description)/meshes/fairino3_v6/forearm_link.STL" />
-      </geometry>
-      <material
-        name="">
-        <color
-          rgba="0.89804 0.91765 0.92941 1" />
-      </material>
-    </visual>
-    <collision>
-      <origin
-        xyz="0 0 0"
-        rpy="0 0 0" />
-      <geometry>
-        <mesh
-          filename="package://fairino_description)/meshes/fairino3_v6/forearm_link.STL" />
-      </geometry>
-    </collision>
-  </link>
+          filename="file://$(find fairino_description)/meshes/fairino3_v6/forearm_link.STL" />
+      </geometry>
+      <material
+        name="">
+        <color
+          rgba="0.89804 0.91765 0.92941 1" />
+      </material>
+    </visual>
+    <collision>
+      <origin
+        xyz="0 0 0"
+        rpy="0 0 0" />
+      <geometry>
+        <mesh
+          filename="file://$(find fairino_description)/meshes/fairino3_v6/forearm_link.STL" />
+      </geometry>
+    </collision>
+  </link>
+  <gazebo reference="${prefix}forearm_link"><self_collide>false</self_collide></gazebo>
   <joint
     name="${prefix}joint3"
@@ -249,4 +276,14 @@
       k_velocity="10" />
   </joint>
+  <transmission name="${prefix}joint3_trans">
+    <type>transmission_interface/SimpleTransmission</type>
+    <joint name="${prefix}joint3">
+      <hardwareInterface>hardware_interface/PositionJointInterface</hardwareInterface>
+    </joint>
+    <actuator name="${prefix}joint3_motor">
+      <hardwareInterface>hardware_interface/PositionJointInterface</hardwareInterface>
+      <mechanicalReduction>1</mechanicalReduction>
+    </actuator>
+  </transmission>
   <link
     name="${prefix}wrist1_link">
@@ -271,22 +308,23 @@
       <geometry>
         <mesh
-          filename="file:///$(find fairino_description)/meshes/fairino3_v6/wrist1_link.STL" />
-      </geometry>
-      <material
-        name="">
-        <color
-          rgba="0.89804 0.91765 0.92941 1" />
-      </material>
-    </visual>
-    <collision>
-      <origin
-        xyz="0 0 0"
-        rpy="0 0 0" />
-      <geometry>
-        <mesh
-          filename="file:///$(find fairino_description)/meshes/fairino3_v6/wrist1_link.STL" />
-      </geometry>
-    </collision>
-  </link>
+          filename="file://$(find fairino_description)/meshes/fairino3_v6/wrist1_link.STL" />
+      </geometry>
+      <material
+        name="">
+        <color
+          rgba="0.89804 0.91765 0.92941 1" />
+      </material>
+    </visual>
+    <collision>
+      <origin
+        xyz="0 0 0"
+        rpy="0 0 0" />
+      <geometry>
+        <mesh
+          filename="file://$(find fairino_description)/meshes/fairino3_v6/wrist1_link.STL" />
+      </geometry>
+    </collision>
+  </link>
+  <gazebo reference="${prefix}wrist1_link"><self_collide>false</self_collide></gazebo>
   <joint
     name="${prefix}joint4"
@@ -318,4 +356,14 @@
       k_velocity="10" />
   </joint>
+  <transmission name="${prefix}joint4_trans">
+    <type>transmission_interface/SimpleTransmission</type>
+    <joint name="${prefix}joint4">
+      <hardwareInterface>hardware_interface/PositionJointInterface</hardwareInterface>
+    </joint>
+    <actuator name="${prefix}joint4_motor">
+      <hardwareInterface>hardware_interface/PositionJointInterface</hardwareInterface>
+      <mechanicalReduction>1</mechanicalReduction>
+    </actuator>
+  </transmission>
   <link
     name="${prefix}wrist2_link">
@@ -340,22 +388,23 @@
       <geometry>
         <mesh
-          filename="file:///$(find fairino_description)/meshes/fairino3_v6/wrist2_link.STL" />
-      </geometry>
-      <material
-        name="">
-        <color
-          rgba="0.89804 0.91765 0.92941 1" />
-      </material>
-    </visual>
-    <collision>
-      <origin
-        xyz="0 0 0"
-        rpy="0 0 0" />
-      <geometry>
-        <mesh
-          filename="file:///$(find fairino_description)/meshes/fairino3_v6/wrist2_link.STL" />
-      </geometry>
-    </collision>
-  </link>
+          filename="file://$(find fairino_description)/meshes/fairino3_v6/wrist2_link.STL" />
+      </geometry>
+      <material
+        name="">
+        <color
+          rgba="0.89804 0.91765 0.92941 1" />
+      </material>
+    </visual>
+    <collision>
+      <origin
+        xyz="0 0 0"
+        rpy="0 0 0" />
+      <geometry>
+        <mesh
+          filename="file://$(find fairino_description)/meshes/fairino3_v6/wrist2_link.STL" />
+      </geometry>
+    </collision>
+  </link>
+  <gazebo reference="${prefix}wrist2_link"><self_collide>false</self_collide></gazebo>
   <joint
     name="${prefix}joint5"
@@ -387,4 +436,14 @@
       k_velocity="10" />
   </joint>
+  <transmission name="${prefix}joint5_trans">
+    <type>transmission_interface/SimpleTransmission</type>
+    <joint name="${prefix}joint5">
+      <hardwareInterface>hardware_interface/PositionJointInterface</hardwareInterface>
+    </joint>
+    <actuator name="${prefix}joint5_motor">
+      <hardwareInterface>hardware_interface/PositionJointInterface</hardwareInterface>
+      <mechanicalReduction>1</mechanicalReduction>
+    </actuator>
+  </transmission>
   <link
     name="${prefix}wrist3_link">
@@ -409,22 +468,23 @@
       <geometry>
         <mesh
-          filename="file:///$(find fairino_description)/meshes/fairino3_v6/wrist3_link.STL" />
-      </geometry>
-      <material
-        name="">
-        <color
-          rgba="0.89804 0.91765 0.92941 1" />
-      </material>
-    </visual>
-    <collision>
-      <origin
-        xyz="0 0 0"
-        rpy="0 0 0" />
-      <geometry>
-        <mesh
-          filename="file:///$(find fairino_description)/meshes/fairino3_v6/wrist3_link.STL" />
-      </geometry>
-    </collision>
-  </link>
+          filename="file://$(find fairino_description)/meshes/fairino3_v6/wrist3_link.STL" />
+      </geometry>
+      <material
+        name="">
+        <color
+          rgba="0.89804 0.91765 0.92941 1" />
+      </material>
+    </visual>
+    <collision>
+      <origin
+        xyz="0 0 0"
+        rpy="0 0 0" />
+      <geometry>
+        <mesh
+          filename="file://$(find fairino_description)/meshes/fairino3_v6/wrist3_link.STL" />
+      </geometry>
+    </collision>
+  </link>
+  <gazebo reference="${prefix}wrist3_link"><self_collide>false</self_collide></gazebo>
   <joint
     name="${prefix}joint6"
@@ -456,4 +516,14 @@
       k_velocity="10" />
   </joint>
+  <transmission name="${prefix}joint6_trans">
+    <type>transmission_interface/SimpleTransmission</type>
+    <joint name="${prefix}joint6">
+      <hardwareInterface>hardware_interface/PositionJointInterface</hardwareInterface>
+    </joint>
+    <actuator name="${prefix}joint6_motor">
+      <hardwareInterface>hardware_interface/PositionJointInterface</hardwareInterface>
+      <mechanicalReduction>1</mechanicalReduction>
+    </actuator>
+  </transmission>
   </xacro:macro>
 </robot>
