Commit message: RViz visualizes dual arms with initial positions, Gazebo simulates dual arms via joint states

File: src/fairino_description/urdf_dual_arms/fairino3_v6_robot.prefixed.urdf.xacro (robot description, xacro)
@@ -24,19 +24,19 @@
       <geometry>
         <mesh
-          filename="file://$(find fairino_description)/meshes/fairino3_v6/base_link.STL" />
-      </geometry>
-      <material
-        name="">
-        <color
-          rgba="0.89804 0.91765 0.92941 1" />
-      </material>
-    </visual>
-    <collision>
-      <origin
-        xyz="0 0 0"
-        rpy="0 0 0" />
-      <geometry>
-        <mesh
-          filename="file://$(find fairino_description)/meshes/fairino3_v6/base_link.STL" />
+          filename="package://fairino_description/meshes/fairino3_v6/base_link.STL" />
+      </geometry>
+      <material
+        name="">
+        <color
+          rgba="0.89804 0.91765 0.92941 1" />
+      </material>
+    </visual>
+    <collision>
+      <origin
+        xyz="0 0 0"
+        rpy="0 0 0" />
+      <geometry>
+        <mesh
+          filename="package://fairino_description/meshes/fairino3_v6/base_link.STL" />
       </geometry>
     </collision>
@@ -68,19 +68,19 @@
       <geometry>
         <mesh
-          filename="file://$(find fairino_description)/meshes/fairino3_v6/shoulder_link.STL" />
-      </geometry>
-      <material
-        name="">
-        <color
-          rgba="0.89804 0.91765 0.92941 1" />
-      </material>
-    </visual>
-    <collision>
-      <origin
-        xyz="0 0 0"
-        rpy="0 0 0" />
-      <geometry>
-        <mesh
-          filename="file://$(find fairino_description)/meshes/fairino3_v6/shoulder_link.STL" />
+          filename="package://fairino_description/meshes/fairino3_v6/shoulder_link.STL" />
+      </geometry>
+      <material
+        name="">
+        <color
+          rgba="0.89804 0.91765 0.92941 1" />
+      </material>
+    </visual>
+    <collision>
+      <origin
+        xyz="0 0 0"
+        rpy="0 0 0" />
+      <geometry>
+        <mesh
+          filename="package://fairino_description/meshes/fairino3_v6/shoulder_link.STL" />
       </geometry>
     </collision>
@@ -148,19 +148,19 @@
       <geometry>
         <mesh
-          filename="file://$(find fairino_description)/meshes/fairino3_v6/upperarm_link.STL" />
-      </geometry>
-      <material
-        name="">
-        <color
-          rgba="0.89804 0.91765 0.92941 1" />
-      </material>
-    </visual>
-    <collision>
-      <origin
-        xyz="0 0 0"
-        rpy="0 0 0" />
-      <geometry>
-        <mesh
-          filename="file://$(find fairino_description)/meshes/fairino3_v6/upperarm_link.STL" />
+          filename="package://fairino_description/meshes/fairino3_v6/upperarm_link.STL" />
+      </geometry>
+      <material
+        name="">
+        <color
+          rgba="0.89804 0.91765 0.92941 1" />
+      </material>
+    </visual>
+    <collision>
+      <origin
+        xyz="0 0 0"
+        rpy="0 0 0" />
+      <geometry>
+        <mesh
+          filename="package://fairino_description/meshes/fairino3_v6/upperarm_link.STL" />
       </geometry>
     </collision>
@@ -228,19 +228,19 @@
       <geometry>
         <mesh
-          filename="file://$(find fairino_description)/meshes/fairino3_v6/forearm_link.STL" />
-      </geometry>
-      <material
-        name="">
-        <color
-          rgba="0.89804 0.91765 0.92941 1" />
-      </material>
-    </visual>
-    <collision>
-      <origin
-        xyz="0 0 0"
-        rpy="0 0 0" />
-      <geometry>
-        <mesh
-          filename="file://$(find fairino_description)/meshes/fairino3_v6/forearm_link.STL" />
+          filename="package://fairino_description/meshes/fairino3_v6/forearm_link.STL" />
+      </geometry>
+      <material
+        name="">
+        <color
+          rgba="0.89804 0.91765 0.92941 1" />
+      </material>
+    </visual>
+    <collision>
+      <origin
+        xyz="0 0 0"
+        rpy="0 0 0" />
+      <geometry>
+        <mesh
+          filename="package://fairino_description/meshes/fairino3_v6/forearm_link.STL" />
       </geometry>
     </collision>
@@ -308,19 +308,19 @@
       <geometry>
         <mesh
-          filename="file://$(find fairino_description)/meshes/fairino3_v6/wrist1_link.STL" />
-      </geometry>
-      <material
-        name="">
-        <color
-          rgba="0.89804 0.91765 0.92941 1" />
-      </material>
-    </visual>
-    <collision>
-      <origin
-        xyz="0 0 0"
-        rpy="0 0 0" />
-      <geometry>
-        <mesh
-          filename="file://$(find fairino_description)/meshes/fairino3_v6/wrist1_link.STL" />
+          filename="package://fairino_description/meshes/fairino3_v6/wrist1_link.STL" />
+      </geometry>
+      <material
+        name="">
+        <color
+          rgba="0.89804 0.91765 0.92941 1" />
+      </material>
+    </visual>
+    <collision>
+      <origin
+        xyz="0 0 0"
+        rpy="0 0 0" />
+      <geometry>
+        <mesh
+          filename="package://fairino_description/meshes/fairino3_v6/wrist1_link.STL" />
       </geometry>
     </collision>
@@ -388,19 +388,19 @@
       <geometry>
         <mesh
-          filename="file://$(find fairino_description)/meshes/fairino3_v6/wrist2_link.STL" />
-      </geometry>
-      <material
-        name="">
-        <color
-          rgba="0.89804 0.91765 0.92941 1" />
-      </material>
-    </visual>
-    <collision>
-      <origin
-        xyz="0 0 0"
-        rpy="0 0 0" />
-      <geometry>
-        <mesh
-          filename="file://$(find fairino_description)/meshes/fairino3_v6/wrist2_link.STL" />
+          filename="package://fairino_description/meshes/fairino3_v6/wrist2_link.STL" />
+      </geometry>
+      <material
+        name="">
+        <color
+          rgba="0.89804 0.91765 0.92941 1" />
+      </material>
+    </visual>
+    <collision>
+      <origin
+        xyz="0 0 0"
+        rpy="0 0 0" />
+      <geometry>
+        <mesh
+          filename="package://fairino_description/meshes/fairino3_v6/wrist2_link.STL" />
       </geometry>
     </collision>
@@ -468,19 +468,19 @@
       <geometry>
         <mesh
-          filename="file://$(find fairino_description)/meshes/fairino3_v6/wrist3_link.STL" />
-      </geometry>
-      <material
-        name="">
-        <color
-          rgba="0.89804 0.91765 0.92941 1" />
-      </material>
-    </visual>
-    <collision>
-      <origin
-        xyz="0 0 0"
-        rpy="0 0 0" />
-      <geometry>
-        <mesh
-          filename="file://$(find fairino_description)/meshes/fairino3_v6/wrist3_link.STL" />
+          filename="package://fairino_description/meshes/fairino3_v6/wrist3_link.STL"/>
+      </geometry>
+      <material
+        name="">
+        <color
+          rgba="0.89804 0.91765 0.92941 1" />
+      </material>
+    </visual>
+    <collision>
+      <origin
+        xyz="0 0 0"
+        rpy="0 0 0" />
+      <geometry>
+        <mesh
+          filename="package://fairino_description/meshes/fairino3_v6/wrist3_link.STL" />
       </geometry>
     </collision>
